Commit message: Final_AMR003

File: description/gazebo_control.xacro (robot description, xacro)
@@ -7,6 +7,6 @@
             <right_joint>right_wheel_joint</right_joint>
             <!-- Kích thước cơ khí từ file CAD của Tiến -->
-            <wheel_separation>0.565</wheel_separation> <!-- Khoảng cách 2 bánh chính (56.5cm) -->
-            <wheel_diameter>0.089</wheel_diameter>     <!-- Đường kính bánh xe (8.9cm) -->
+            <wheel_separation>0.572</wheel_separation>
+            <wheel_diameter>0.074</wheel_diameter>    <!-- Đường kính bánh xe (8.9cm) -->
             <!-- Giới hạn lực động cơ -->
             <max_wheel_torque>20</max_wheel_torque>
@@ -17,5 +17,5 @@
             <publish_odom>true</publish_odom>
             <publish_odom_tf>true</publish_odom_tf>
-            <publish_wheel_tf>true</publish_wheel_tf>
+            <publish_wheel_tf>false</publish_wheel_tf>
         </plugin>
     </gazebo>

File: description/lidar.xacro (robot description, xacro)
@@ -1,29 +1,34 @@
 <?xml version="1.0"?>
-<robot xmlns:xacro="http://www.ros.org/wiki/xacro" >
+<robot xmlns:xacro="http://www.ros.org/wiki/xacro">
     <joint name="laser_joint" type="fixed">
-        <origin xyz="0.072995 0 0.45" rpy="0 0 0" />
-        <parent link="base_link" />
-        <child link="laser_frame" />
+        <!-- Vị trí lấy từ URDF SolidWorks mới (lidar_joint) -->
+        <!-- x=0.057994, y≈0, z=0.5808 so với base_link -->
+        <origin xyz="-0.00063688 0.00045389 0.58047" rpy="0 0 0"/>
+        <parent link="base_link"/>
+        <child link="laser_frame"/>
     </joint>
     <link name="laser_frame">
         <inertial>
-            <origin xyz="1.6653E-16 -1.4832E-18 -0.031831" rpy="0 0 0" />
-            <mass value="0.4" />
-            <inertia ixx="0.00085342" ixy="-7.7037E-34" ixz="-2.3908E-18"
-                     iyy="0.00085342" iyz="1.6803E-20" izz="0.0015382" />
+            <origin xyz="0 0 0" rpy="0 0 0"/>
+            <mass value="0.2"/>
+            <inertia
+                ixx="0.001" ixy="0" ixz="0"
+                iyy="0.001" iyz="0"
+                izz="0.001"/>
         </inertial>
         <visual>
-            <!-- Sử dụng hình trụ thay thế cho file .STL để hiển thị tạm thời -->
-            <origin xyz="0 0 0" rpy="0 0 0" />
+            <origin xyz="0 0 0" rpy="0 0 0"/>
             <geometry>
-                <cylinder radius="0.05" length="0.04"/>
+                <!-- Dùng mesh STL từ SolidWorks export -->
+                <mesh filename="package://amr_003/meshes/lidar_link.STL"/>
             </geometry>
-            <material name="laser_color">
-                <color rgba="0.79216 0.81961 0.93333 1" />
+            <material name="">
+                <color rgba="0.2 0.2 0.2 1"/>
             </material>
         </visual>
         <collision>
-            <origin xyz="0 0 0" rpy="0 0 0" />
+            <origin xyz="0 0 0" rpy="0 0 0"/>
             <geometry>
+                <!-- Dùng cylinder đơn giản cho collision (nhanh hơn mesh) -->
                 <cylinder radius="0.05" length="0.04"/>
             </geometry>
@@ -33,18 +38,18 @@
         <material>Gazebo/Black</material>
         <sensor name="laser" type="ray">
-            <pose> 0 0 0 0 0 0 </pose>
+            <pose>0 0 0 0 0 0</pose>
             <visualize>false</visualize>
-            <update_rate>10</update_rate>
+            <update_rate>10.0</update_rate>
             <ray>
                 <scan>
                     <horizontal>
                         <samples>360</samples>
-                        <min_angle>-3.14</min_angle>
-                        <max_angle>3.14</max_angle>
+                        <min_angle>-3.14159</min_angle>
+                        <max_angle>3.14159</max_angle>
                     </horizontal>
                 </scan>
                 <range>
                     <min>0.3</min>
-                    <max>12</max>
+                    <max>12.0</max>
                 </range>
             </ray>

File: description/robot.urdf.xacro (robot description, xacro)
@@ -2,4 +2,5 @@
 <robot xmlns:xacro="http://www.ros.org/wiki/xacro" name="amr_003">
     <xacro:arg name="use_ros2_control" default="true"/>
+    <xacro:arg name="sim_mode" default="true"/>
     <xacro:include filename="robot_core.xacro" />
     <xacro:if value="$(arg use_ros2_control)">

File: description/robot_core.xacro (robot description, xacro)
@@ -1,194 +1,180 @@
 <?xml version="1.0"?>
-<robot xmlns:xacro="http://www.ros.org/wiki/xacro" >
+<robot xmlns:xacro="http://www.ros.org/wiki/xacro">
     <xacro:include filename="inertial_macros.xacro"/>
-    <material name="white">
-        <color rgba="1 1 1 1" />
-    </material>
-    <material name="black">
-        <color rgba="0.1 0.1 0.1 1" />
-    </material>
-    <material name="transparent_white">
-        <color rgba="0.79216 0.81961 0.93333 0.6" />
-    </material>
-    <!-- ========================================== -->
-    <!-- GỐC ROBOT (BASE FOOTPRINT) -->
-    <!-- ========================================== -->
-    <link name="base_footprint"></link>
+    <material name="white"><color rgba="1 1 1 1" /></material>
+    <material name="black"><color rgba="0.1 0.1 0.1 1" /></material>
+    <material name="transparent_white"><color rgba="0.79216 0.81961 0.93333 0.6" /></material>
+    <link name="base_footprint"/>
     <joint name="base_footprint_joint" type="fixed">
         <parent link="base_footprint"/>
         <child link="base_link"/>
-        <origin xyz="0.1451 0 0.089" rpy="0 0 0"/>
+        <origin xyz="0 0 0.0445" rpy="0 0 0"/>
     </joint>
-    <!-- ========================================== -->
-    <!-- KHUNG XE CHÍNH (BASE LINK - NẶNG 6KG) -->
-    <!-- ========================================== -->
     <link name="base_link">
         <inertial>
-            <origin xyz="-0.0055205 -4.5468E-17 0.02" rpy="0 0 0" />
-            <mass value="10" />
-            <inertia ixx="0.08" ixy="0" ixz="0" iyy="0.12" iyz="0" izz="0.16" />
+            <origin xyz="0.106814398044022 0 0.057" rpy="0 0 0"/>
+            <mass value="3.2625"/>
+            <inertia ixx="0.056906796875" ixy="0" ixz="0" iyy="0.0609283294420498" iyz="0" izz="0.11771278256705"/>
         </inertial>
         <visual>
-            <origin xyz="0 0 0" rpy="0 0 0" />
-            <geometry>
-                <mesh filename="package://amr_003/meshes/base_link.STL" />
-            </geometry>
+            <origin xyz="0 0 0" rpy="0 0 0"/>
+            <geometry><mesh filename="package://amr_003/meshes/base_link.STL"/></geometry>
             <material name="transparent_white"/>
         </visual>
         <collision>
-            <!-- Dùng hộp đơn giản cho va chạm Chassis để Gazebo tính toán mượt nhẹ -->
-            <origin xyz="0 0 0.1" rpy="0 0 0" />
-            <geometry>
-                <box size="0.45 0.35 0.2"/>
-            </geometry>
+            <origin xyz="0 0 0.15" rpy="0 0 0"/>
+            <geometry><box size="0.45 0.35 0.1"/></geometry>
         </collision>
     </link>
-    <!-- ========================================== -->
-    <!-- BÁNH XE DẪN ĐỘNG TRÁI -->
-    <!-- ========================================== -->
-    <link name="left_wheel">
+    <link name="chassis_link">
         <inertial>
-            <origin xyz="2.7756E-17 3.4694E-18 -0.01" rpy="0 0 0" />
-            <mass value="0.1415" />
-            <inertia ixx="7.859E-05" ixy="0" ixz="0" iyy="7.859E-05" iyz="0" izz="0.00014084" />
+            <origin xyz="0.222980078166213 0 0.05" rpy="0 0 0" />
+            <mass value="7.00166781646683" />
+            <inertia ixx="0.109362090239879" ixy="0" ixz="0.00489513284151782" iyy="0.11176801072697" iyz="0" izz="0.208620108039956" />
         </inertial>
         <visual>
-            <origin xyz="0 0 0" rpy="0 0 0" />
-            <geometry>
-                <mesh filename="package://amr_003/meshes/left_wheel.STL" />
-            </geometry>
+            <origin xyz="0 0 0" rpy="0 0 0"/>
+            <geometry><mesh filename="package://amr_003/meshes/chassis_link.STL"/></geometry>
+            <material name="transparent_white"/>
+        </visual>
+    </link>
+    <joint name="chassis_joint" type="fixed">
+        <origin xyz="-0.12372 0 0.0345" rpy="0 0 0"/>
+        <parent link="base_link"/>
+        <child link="chassis_link"/>
+    </joint>
+    <link name="left_wheel_link">
+        <inertial>
+            <origin xyz="0 0 0" rpy="0 0 0"/>
+            <mass value="1.0"/>
+            <inertia ixx="0.001" ixy="0" ixz="0" iyy="0.001" iyz="0" izz="0.001" />
+        </inertial>
+        <visual>
+            <origin xyz="0 0 0" rpy="0 0 0"/>
+            <geometry><mesh filename="package://amr_003/meshes/left_wheel_link.STL"/></geometry>
             <material name="black"/>
         </visual>
         <collision>
-            <origin xyz="0 0 0" rpy="0 0 0" />
-            <geometry>
-                <sphere radius="0.0445" />
-                <!-- length="0.04" -->
-            </geometry>
+            <origin xyz="0 0 0" rpy="0 0 0"/>
+            <geometry><sphere radius="0.037"/></geometry>
         </collision>
     </link>
     <joint name="left_wheel_joint" type="continuous">
-        <origin xyz="-0.1451 0.2825 -0.0445" rpy="-1.5708 0 0" />
-        <parent link="base_link" />
-        <child link="left_wheel" />
-        <axis xyz="0 0 1" />
-        <dynamics damping="0.1" friction="0.1" />
+        <origin xyz="0 0.286 -0.0075" rpy="-1.5708 0 0"/>
+        <parent link="base_link"/>
+        <child link="left_wheel_link"/>
+        <axis xyz="0 0 1"/>
+        <limit effort="10.0" velocity="20.0"/>
     </joint>
-    <!-- ========================================== -->
-    <!-- BÁNH XE DẪN ĐỘNG PHẢI -->
-    <!-- ========================================== -->
-    <link name="right_wheel">
+    <link name="right_wheel_link">
         <inertial>
-            <origin xyz="-4.1633E-17 -3.4694E-18 0.01" rpy="0 0 0" />
-            <mass value="0.1415" />
-            <inertia ixx="7.859E-05" ixy="0" ixz="0" iyy="7.859E-05" iyz="0" izz="0.00014084" />
+            <origin xyz="0 0 0" rpy="0 0 0"/>
+            <mass value="1.0"/>
+            <inertia ixx="0.001" ixy="0" ixz="0" iyy="0.001" iyz="0" izz="0.001" />
         </inertial>
         <visual>
-            <origin xyz="0 0 0" rpy="0 0 0" />
-            <geometry>
-                <mesh filename="package://amr_003/meshes/right_wheel.STL" />
-            </geometry>
+            <origin xyz="0 0 0" rpy="0 0 0"/>
+            <geometry><mesh filename="package://amr_003/meshes/right_wheel_link.STL"/></geometry>
             <material name="black"/>
         </visual>
         <collision>
-            <origin xyz="0 0 0" rpy="0 0 0" />
-            <geometry>
-                <sphere radius="0.0445" />
-            </geometry>
+            <origin xyz="0 0 0" rpy="0 0 0"/>
+            <geometry><sphere radius="0.037"/></geometry>
         </collision>
     </link>
     <joint name="right_wheel_joint" type="continuous">
-        <origin xyz="-0.1451 -0.2825 -0.0445" rpy="-1.5708 0 0" />
-        <parent link="base_link" />
-        <child link="right_wheel" />
-        <axis xyz="0 0 1" />
-        <dynamics damping="0.1" friction="0.1" />
+        <origin xyz="0 -0.286 -0.0075" rpy="-1.5708 0 0"/>
+        <parent link="base_link"/>
+        <child link="right_wheel_link"/>
+        <axis xyz="0 0 1"/>
+        <limit effort="10.0" velocity="20.0"/>
     </joint>
-    <!-- ========================================== -->
-    <!-- CỔ XOAY CASTER BRACKET (PHUỘC TRƯỚC) -->
-    <!-- ========================================== -->
-    <link name="caster_wheel_1">
-        <inertial>
-            <origin xyz="1.6653E-16 1.2291E-17 -0.013121" rpy="0 0 0" />
-            <mass value="0.5" />
-            <inertia ixx="0.001" ixy="0" ixz="0" iyy="0.001" iyz="0" izz="0.001" />
-        </inertial>
+    <link name="bracker_link">
         <visual>
-            <origin xyz="0 0 0" rpy="0 0 0" />
-            <geometry>
-                <mesh filename="package://amr_003/meshes/caster_wheel_1.STL" />
-            </geometry>
+            <origin xyz="0 0 0" rpy="0 0 0"/>
+            <geometry><mesh filename="package://amr_003/meshes/bracker_link.STL"/></geometry>
             <material name="black"/>
         </visual>
+    </link>
+    <joint name="bracker_joint" type="fixed">
+        <origin xyz="0.35672 -0.00047549 0.0245" rpy="0 0 0"/>
+        <parent link="base_link"/>
+        <child link="bracker_link"/>
+    </joint>
+    <link name="caster_wheel_link">
+        <visual>
+            <origin xyz="0 0 0" rpy="0 0 0"/>
+            <geometry><mesh filename="package://amr_003/meshes/caster_wheel_link.STL"/></geometry>
+            <material name="black"/>
+        </visual>
+    </link>
+    <joint name="caster_wheel_joint" type="fixed">
+        <origin xyz="0 0.00047549 -0.043" rpy="-1.5708 0 0"/>
+        <parent link="bracker_link"/>
+        <child link="caster_wheel_link"/>
+    </joint>
+    <link name="front_caster_collision_link">
+        <inertial>
+            <origin xyz="0 0 0" rpy="0 0 0"/>
+            <mass value="3.0"/>
+            <inertia ixx="0.01" ixy="0" ixz="0" iyy="0.01" iyz="0" izz="0.01"/>
+        </inertial>
         <collision>
-            <origin xyz="0 0 -0.015" rpy="0 0 0" />
-            <geometry>
-                <box size="0.03 0.03 0.02"/>
-            </geometry>
+            <origin xyz="0 0 0" rpy="0 0 0"/>
+            <geometry><sphere radius="0.026"/></geometry>
         </collision>
     </link>
-    <joint name="caster_bracket_joint" type="fixed">
-        <origin xyz="0.23009 0 -0.015" rpy="0 0 0" />
-        <parent link="base_link" />
-        <child link="caster_wheel_1" />
-        <axis xyz="0 0 1" />
-        <dynamics damping="0.1" friction="0.1" /> <!-- Đã giảm damping để mượt hơn -->
+    <joint name="front_caster_collision_joint" type="fixed">
+        <origin xyz="0.415 0 -0.0185" rpy="0 0 0"/>
+        <parent link="base_link"/>
+        <child link="front_caster_collision_link"/>
     </joint>
-    <!-- ========================================== -->
-    <!-- BÁNH XE CASTER TRƯỚC (QUAY TỰ DO) -->
-    <!-- ========================================== -->
-    <link name="caster_wheel_2">
+    <link name="rear_caster_collision_link">
         <inertial>
-            <origin xyz="-5.5511E-17 -5.5511E-17 -6.7405E-19" rpy="0 0 0" />
-            <mass value="0.5" />
-            <inertia ixx="0.001" ixy="0" ixz="0" iyy="0.001" iyz="0" izz="0.001" />
+            <origin xyz="0 0 0" rpy="0 0 0"/>
+            <mass value="1.0"/>
+            <inertia ixx="0.01" ixy="0" ixz="0" iyy="0.01" iyz="0" izz="0.01"/>
         </inertial>
-        <visual>
-            <origin xyz="0 0 0" rpy="0 0 0" />
-            <geometry>
-                <mesh filename="package://amr_003/meshes/caster_wheel_2.STL" />
-            </geometry>
-            <material name="black"/>
-        </visual>
         <collision>
-            <origin xyz="0 0 0" rpy="0 0 0" />
-            <geometry>
-                <sphere radius="0.026" />
-            </geometry>
+            <origin xyz="0 0 0" rpy="0 0 0"/>
+            <geometry><sphere radius="0.026"/></geometry>
         </collision>
     </link>
-    <joint name="caster_wheel_joint" type="fixed">
-        <origin xyz="0 0 -0.048" rpy="-1.5708 0 0" />
-        <parent link="caster_wheel_1" />
-        <child link="caster_wheel_2" />
-        <axis xyz="0 0 1" />
-        <dynamics damping="0.1" friction="0.1" />
+    <joint name="rear_caster_collision_joint" type="fixed">
+        <origin xyz="-0.35 0 -0.0185" rpy="0 0 0"/>
+        <parent link="base_link"/>
+        <child link="rear_caster_collision_link"/>
     </joint>
-    <!-- ========================================== -->
-    <!-- CẤU HÌNH VẬT LÝ GAZEBO ĐẶC THÙ -->
-    <!-- ========================================== -->
-    <gazebo reference="base_link">
-        <material>Gazebo/Orange</material>
-    </gazebo>
-    <gazebo reference="left_wheel">
-        <mu1>2.0</mu1>
-        <mu2>2.0</mu2>
+    <gazebo reference="base_link"><material>Gazebo/Orange</material></gazebo>
+    <gazebo reference="chassis_link"><material>Gazebo/Grey</material></gazebo>
+    <gazebo reference="left_wheel_link">
+        <mu1>1.5</mu1> <mu2>1.5</mu2>
+        <kp>1000000.0</kp>
+        <kd>100.0</kd>
+        <minDepth>0.001</minDepth>
+        <maxVel>0.0</maxVel>
         <material>Gazebo/FlatBlack</material>
     </gazebo>
-    <gazebo reference="right_wheel">
-        <mu1>2.0</mu1>
-        <mu2>2.0</mu2>
+    <gazebo reference="right_wheel_link">
+        <mu1>1.5</mu1> <mu2>1.5</mu2>
+        <kp>1000000.0</kp>
+        <kd>100.0</kd>
+        <minDepth>0.001</minDepth>
+        <maxVel>0.0</maxVel>
         <material>Gazebo/FlatBlack</material>
     </gazebo>
-    <gazebo reference="caster_wheel_1">
-        <material>Gazebo/Grey</material>
+    <gazebo reference="front_caster_collision_link">
+        <mu1>0.0</mu1> <mu2>0.0</mu2>
+        <kp>1000000.0</kp>
+        <kd>100.0</kd>
+        <minDepth>0.001</minDepth>
+        <maxVel>0.0</maxVel>
     </gazebo>
-    <gazebo reference="caster_wheel_2">
-        <mu1>0.0</mu1>
-        <mu2>0.0</mu2>
-        <kp>10000000.0</kp>
-        <kd>1.0</kd>
+    <gazebo reference="rear_caster_collision_link">
+        <mu1>0.0</mu1> <mu2>0.0</mu2>
+        <kp>1000000.0</kp>
+        <kd>100.0</kd>
         <minDepth>0.001</minDepth>
-        <material>Gazebo/Black</material>
+        <maxVel>0.0</maxVel>
     </gazebo>
 </robot>

File: description/ros2_control.xacro (robot description, xacro)
@@ -1,57 +1,62 @@
 <?xml version="1.0"?>
 <robot xmlns:xacro="http://www.ros.org/wiki/xacro">
-    <ros2_control name="RealRobot" type="system">
-        <hardware>
-            <plugin>diffdrive_arduino/DiffDriveArduinoHardware</plugin>
-            <param name="left_wheel_name">left_wheel_joint</param>
-            <param name="right_wheel_name">right_wheel_joint</param>
-            <param name="loop_rate">30</param>
-            <param name="device">/dev/ttyUSB0</param>
-            <param name="baud_rate">57600</param>
-            <param name="timeout_ms">1000</param>
-            <param name="enc_counts_per_rev">342</param>
-        </hardware>
-        <joint name="left_wheel_joint">
-            <command_interface name="velocity">
-                <param name="min">-20</param>
-                <param name="max">20</param>
-            </command_interface>
-            <state_interface name="position"/>
-            <state_interface name="velocity"/>
-        </joint>
-        <joint name="right_wheel_joint">
-            <command_interface name="velocity">
-                <param name="min">-20</param>
-                <param name="max">20</param>
-            </command_interface>
-            <state_interface name="position"/>
-            <state_interface name="velocity"/>
-        </joint>
-    </ros2_control>
-    <!-- <ros2_control name="GazeboSystem" type="system">
-        <hardware>
-            <plugin>gazebo_ros2_control/GazeboSystem</plugin>
-        </hardware>
-        <joint name="left_wheel_joint">
-            <command_interface name="velocity">
-                <param name="min">-20</param>
-                <param name="max">20</param>
-            </command_interface>
-            <state_interface name="velocity"/>
-            <state_interface name="position"/>
-        </joint>
-        <joint name="right_wheel_joint">
-            <command_interface name="velocity">
-                <param name="min">-20</param>
-                <param name="max">20</param>
-            </command_interface>
-            <state_interface name="velocity"/>
-            <state_interface name="position"/>
-        </joint>
-    </ros2_control> -->
+    <xacro:unless value="$(arg sim_mode)">
+        <ros2_control name="RealRobot" type="system">
+            <hardware>
+                <plugin>diffdrive_arduino/DiffDriveArduinoHardware</plugin>
+                <param name="left_wheel_name">left_wheel_joint</param>
+                <param name="right_wheel_name">right_wheel_joint</param>
+                <param name="loop_rate">30</param>
+                <param name="device">/dev/ttyUSB0</param>
+                <param name="baud_rate">57600</param>
+                <param name="timeout_ms">1000</param>
+                <param name="enc_counts_per_rev">342</param>
+            </hardware>
+            <joint name="left_wheel_joint">
+                <command_interface name="velocity">
+                    <param name="min">-20</param>
+                    <param name="max">20</param>
+                </command_interface>
+                <state_interface name="position"/>
+                <state_interface name="velocity"/>
+            </joint>
+            <joint name="right_wheel_joint">
+                <command_interface name="velocity">
+                    <param name="min">-20</param>
+                    <param name="max">20</param>
+                </command_interface>
+                <state_interface name="position"/>
+                <state_interface name="velocity"/>
+            </joint>
+        </ros2_control>
+    </xacro:unless>
+    <xacro:if value="$(arg sim_mode)">
+        <ros2_control name="GazeboSystem" type="system">
+            <hardware>
+                <plugin>gazebo_ros2_control/GazeboSystem</plugin>
+            </hardware>
+            <joint name="left_wheel_joint">
+                <command_interface name="velocity">
+                    <param name="min">-20</param>
+                    <param name="max">20</param>
+                </command_interface>
+                <state_interface name="position"/>
+                <state_interface name="velocity"/>
+            </joint>
+            <joint name="right_wheel_joint">
+                <command_interface name="velocity">
+                    <param name="min">-20</param>
+                    <param name="max">20</param>
+                </command_interface>
+                <state_interface name="position"/>
+                <state_interface name="velocity"/>
+            </joint>
+        </ros2_control>
     <gazebo>
         <plugin name="gazebo_ros2_control" filename="libgazebo_ros2_control.so">
             <parameters>$(find amr_003)/config/my_controllers.yaml</parameters>
+            <parameters>$(find amr_003)/config/gaz_ros2_ctl_use_sim.yaml</parameters>
         </plugin>
     </gazebo>
+    </xacro:if>
 </robot>
